File: hardware/project-julie-bed-lights.kicad_pcb (KiCad board)
At the start: 2 copper layers, 58 x 60 mm, 27 parts, among them J1 2199230-4, J2 BM06B-SRSS-TB(LF)(SN), J3 Screw_Terminal_01x04, J4 Screw_Terminal_01x02, Q1 IRF8736TRPBF‎, Q2 IRF8736TRPBF‎, Q3 IRF8736TRPBF‎, SW1 SW_SPST, U1 AP63300WU-7

Commit message: Add screw terminal marking
Other:
- board text added: "12V"
- board text added: "B"
- board text added: "G"
- board text added: "GND"
- board text added: "R"
